File: I2C_PINOUT.kicad_sch (KiCad schematic)
At the start: 1 part

Commit message: assign footprints
Parts:
- I2C_PINOUT8: renamed from I2C_PINOUT; footprint (none) -> Connector_PinSocket_1.00mm:PinSocket_1x04_P1.00mm_Vertical
Changed lines of the file:
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@@
 		(dnp no)
 		(fields_autoplaced yes)
-		(property "Reference" "I2C_PINOUT"
+		(property "Reference" "I2C_PINOUT8"
 			(at 162.56 85.0899 0)
 			(effects
@@
 			)
 		)
-		(property "Footprint" ""
+		(property "Footprint" "Connector_PinSocket_1.00mm:PinSocket_1x04_P1.00mm_Vertical"
 			(at 160.02 85.09 0)
 			(effects
@@
 				)
 				(path "/3c2fce68-ba60-4bda-a294-ddd60ff77106/6d11c068-6d98-437f-8725-9d48a876a04d"
-					(reference "I2C_PINOUT")
+					(reference "I2C_PINOUT13")
 					(unit 1)
 				)
@@
 		(dnp no)
 		(fields_autoplaced yes)
-		(property "Reference" "#PWR025"
+		(property "Reference" "#PWR068"
 			(at 148.59 90.17 0)
 			(effects
@@
 		(dnp no)
 		(fields_autoplaced yes)
-		(property "Reference" "#PWR022"
+		(property "Reference" "#PWR067"
 			(at 158.75 87.63 0)
 			(effects

Commit message: start work on pcb design
Parts:
- I2C_PINOUT8: footprint Connector_PinSocket_1.00mm:PinSocket_1x04_P1.00mm_Vertical -> Connector_PinSocket_2.54mm:PinSocket_1x04_P2.54mm_Vertical
Changed lines of the file:
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@@
 			)
 		)
-		(property "Footprint" "Connector_PinSocket_1.00mm:PinSocket_1x04_P1.00mm_Vertical"
+		(property "Footprint" "Connector_PinSocket_2.54mm:PinSocket_1x04_P2.54mm_Vertical"
 			(at 160.02 85.09 0)
 			(effects
@@
 				)
 				(path "/3c2fce68-ba60-4bda-a294-ddd60ff77106/6d11c068-6d98-437f-8725-9d48a876a04d"
-					(reference "I2C_PINOUT13")
+					(reference "I2C_PINOUT0")
 					(unit 1)
 				)
