File: shadow.kicad_sch (KiCad schematic)
At the start: 12 parts, among them SW1 SW_Push, SW2 SW_Push

Commit message: assign footprints
Parts:
- GPIO_L1: renamed from GPIO_L; footprint (none) -> Connector_PinSocket_1.00mm:PinSocket_1x15_P1.00mm_Vertical
- GPIO_R1: renamed from GPIO_R; footprint (none) -> Connector_PinSocket_1.00mm:PinSocket_1x15_P1.00mm_Vertical
- MOTOR_CONN1: renamed from MOTOR_CONN; footprint (none) -> Connector_PinSocket_1.00mm:PinSocket_1x02_P1.00mm_Vertical
- OLED_CONN1: footprint (none) -> Connector_PinSocket_1.00mm:PinSocket_1x04_P1.00mm_Vertical
- PICO_L1: renamed from PICO_L; footprint (none) -> Connector_PinSocket_1.00mm:PinSocket_1x15_P1.00mm_Vertical
- PICO_R1: renamed from PICO_R; footprint (none) -> Connector_PinSocket_1.00mm:PinSocket_1x15_P1.00mm_Vertical
- SENSOR_CONN1: renamed from SENSOR_CONN; footprint (none) -> Connector_PinSocket_1.00mm:PinSocket_1x04_P1.00mm_Vertical
- UART1: footprint (none) -> Connector_PinHeader_1.00mm:PinHeader_1x03_P1.00mm_Vertical
- US_SENSOR_CONN1: renamed from US_SENSOR_CONN; footprint (none) -> Connector_PinHeader_1.00mm:PinHeader_1x04_P1.00mm_Vertical
- renumbered RST_SW to RST_SW1
Changed lines of the file:
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@@
 		(dnp no)
 		(fields_autoplaced yes)
-		(property "Reference" "MOTOR_CONN"
+		(property "Reference" "MOTOR_CONN1"
 			(at 81.28 101.6001 0)
 			(effects
@@
 			)
 		)
-		(property "Footprint" ""
+		(property "Footprint" "Connector_PinSocket_1.00mm:PinSocket_1x02_P1.00mm_Vertical"
 			(at 83.82 101.6 0)
 			(effects
@@
 			(project ""
 				(path "/3c2fce68-ba60-4bda-a294-ddd60ff77106"
-					(reference "MOTOR_CONN")
+					(reference "MOTOR_CONN1")
 					(unit 1)
 				)
@@
 			)
 		)
-		(property "Footprint" ""
+		(property "Footprint" "Connector_PinHeader_1.00mm:PinHeader_1x03_P1.00mm_Vertical"
 			(at 97.79 93.98 0)
 			(effects
@@
 		(on_board yes)
 		(dnp no)
-		(property "Reference" "GPIO_R"
+		(property "Reference" "GPIO_R1"
 			(at 39.624 127.254 0)
 			(effects
@@
 			)
 		)
-		(property "Footprint" ""
+		(property "Footprint" "Connector_PinSocket_1.00mm:PinSocket_1x15_P1.00mm_Vertical"
 			(at 39.37 102.87 0)
 			(effects
@@
 			(project "shadow"
 				(path "/3c2fce68-ba60-4bda-a294-ddd60ff77106"
-					(reference "GPIO_R")
+					(reference "GPIO_R1")
 					(unit 1)
 				)
@@
 		(on_board yes)
 		(dnp no)
-		(property "Reference" "RST_SW"
+		(property "Reference" "RST_SW1"
 			(at 155.956 108.966 0)
 			(effects
@@
 			(project "shadow"
 				(path "/3c2fce68-ba60-4bda-a294-ddd60ff77106"
-					(reference "RST_SW")
+					(reference "RST_SW1")
 					(unit 1)
 				)
@@
 		(dnp no)
 		(fields_autoplaced yes)
-		(property "Reference" "GPIO_L"
+		(property "Reference" "GPIO_L1"
 			(at 26.67 127 0)
 			(effects
@@
 			)
 		)
-		(property "Footprint" ""
+		(property "Footprint" "Connector_PinSocket_1.00mm:PinSocket_1x15_P1.00mm_Vertical"
 			(at 26.67 102.87 0)
 			(effects
@@
 			(project "shadow"
 				(path "/3c2fce68-ba60-4bda-a294-ddd60ff77106"
-					(reference "GPIO_L")
+					(reference "GPIO_L1")
 					(unit 1)
 				)
@@
 		(dnp no)
 		(fields_autoplaced yes)
-		(property "Reference" "PICO_R"
+		(property "Reference" "PICO_R1"
 			(at 128.27 85.09 0)
 			(effects
@@
 			)
 		)
-		(property "Footprint" ""
+		(property "Footprint" "Connector_PinSocket_1.00mm:PinSocket_1x15_P1.00mm_Vertical"
 			(at 128.27 109.22 0)
 			(effects
@@
 			(project "shadow"
 				(path "/3c2fce68-ba60-4bda-a294-ddd60ff77106"
-					(reference "PICO_R")
+					(reference "PICO_R1")
 					(unit 1)
 				)
@@
 		(on_board yes)
 		(dnp no)
-		(property "Reference" "PICO_L"
+		(property "Reference" "PICO_L1"
 			(at 109.728 85.09 0)
 			(effects
@@
 			)
 		)
-		(property "Footprint" ""
+		(property "Footprint" "Connector_PinSocket_1.00mm:PinSocket_1x15_P1.00mm_Vertical"
 			(at 114.3 109.22 0)
 			(effects
@@
 			(project ""
 				(path "/3c2fce68-ba60-4bda-a294-ddd60ff77106"
-					(reference "PICO_L")
+					(reference "PICO_L1")
 					(unit 1)
 				)
@@
 		(dnp no)
 		(fields_autoplaced yes)
-		(property "Reference" "SENSOR_CONN"
+		(property "Reference" "SENSOR_CONN1"
 			(at 238.76 99.0599 0)
 			(effects
@@
 			)
 		)
-		(property "Footprint" ""
+		(property "Footprint" "Connector_PinSocket_1.00mm:PinSocket_1x04_P1.00mm_Vertical"
 			(at 236.22 99.06 0)
 			(effects
@@
 			(project "shadow"
 				(path "/3c2fce68-ba60-4bda-a294-ddd60ff77106"
-					(reference "SENSOR_CONN")
+					(reference "SENSOR_CONN1")
 					(unit 1)
 				)
@@
 			)
 		)
-		(property "Footprint" ""
+		(property "Footprint" "Connector_PinSocket_1.00mm:PinSocket_1x04_P1.00mm_Vertical"
 			(at 236.22 85.09 0)
 			(effects
@@
 		(dnp no)
 		(fields_autoplaced yes)
-		(property "Reference" "US_SENSOR_CONN"
+		(property "Reference" "US_SENSOR_CONN1"
 			(at 238.76 113.0299 0)
 			(effects
@@
 			)
 		)
-		(property "Footprint" ""
+		(property "Footprint" "Connector_PinHeader_1.00mm:PinHeader_1x04_P1.00mm_Vertical"
 			(at 236.22 113.03 0)
 			(effects
@@
 			(project "shadow"
 				(path "/3c2fce68-ba60-4bda-a294-ddd60ff77106"
-					(reference "US_SENSOR_CONN")
-					(unit 1)
-				)
+					(reference "US_SENSOR_CONN1")
+					(unit 1)
+				)

Commit message: start work on pcb design
Parts:
- GPIO_L1, GPIO_R1, PICO_L1, PICO_R1: footprint Connector_PinSocket_1.00mm:PinSocket_1x15_P1.00mm_Vertical -> Connector_PinSocket_2.54mm:PinSocket_1x15_P2.54mm_Vertical
- MOTOR_CONN1: footprint Connector_PinSocket_1.00mm:PinSocket_1x02_P1.00mm_Vertical -> Connector_PinSocket_2.54mm:PinSocket_1x02_P2.54mm_Vertical
- OLED_CONN1, SENSOR_CONN1: footprint Connector_PinSocket_1.00mm:PinSocket_1x04_P1.00mm_Vertical -> Connector_PinSocket_2.54mm:PinSocket_1x04_P2.54mm_Vertical
- RST_SW1, SW1, SW2: footprint Button_Switch_THT:SW_PUSH-12mm -> Button_Switch_THT:SW_PUSH_6mm
- UART1: footprint Connector_PinHeader_1.00mm:PinHeader_1x03_P1.00mm_Vertical -> Connector_PinSocket_2.54mm:PinSocket_1x03_P2.54mm_Vertical
- US_SENSOR_CONN1: footprint Connector_PinHeader_1.00mm:PinHeader_1x04_P1.00mm_Vertical -> Connector_PinSocket_2.54mm:PinSocket_1x04_P2.54mm_Vertical
Connections:
- net GND: now also OLED_CONN1.2 (Pin_2); no longer OLED_CONN1.4 (Pin_4)
- net OLED_SCL: now also OLED_CONN1.3 (Pin_3); no longer OLED_CONN1.2 (Pin_2)
- net OLED_SDA: now also OLED_CONN1.4 (Pin_4); no longer OLED_CONN1.1 (Pin_1)
- net VCC: now also OLED_CONN1.1 (Pin_1); no longer OLED_CONN1.3 (Pin_3)

Commit message: switch to new (better) lipo charger design
Other:
- sheet battery ports: added OUT, OUT_GND; removed 5V, GND
Changed lines of the file:
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@@
 			)
 		)
-		(pin "GND" passive
+		(pin "OUT" input
 			(at 86.36 44.45 270)
 			(effects
@@
 			)
 		)
-		(pin "5V" passive
+		(pin "OUT_GND" input
 			(at 78.74 44.45 270)
 			(effects
