File: shadow.kicad_pcb (KiCad board)
At the start: 2 copper layers, 69.8 x 78.7 mm, 100 parts, among them IC2 XB8089D, J1 USB_C_Receptacle, SW1 SW_Push, SW2 SW_Push, SW3 SW_SPST, U1 TCA9548APWR, U2 TCA9548APWR, U3 BQ24092DGQR, U4 TPS61085DGKR, U5 TPS259621DDAT

Commit message: route pcb
Routing:
- net GND: track 0.00 -> 572.3 mm, vias 0 -> 5
- net VCC: track 0.00 -> 321.5 mm, vias 0 -> 4
- net /battery/BAT+: track 0.00 -> 137.3 mm, vias 0 -> 3
- net Net-(SW3-B): track 0.00 -> 134.9 mm, vias 0 -> 5
- net /battery/BAT-: track 0.00 -> 94.3 mm, vias 0 -> 1
- net Net-(U3-IN): track 0.00 -> 86.7 mm, vias 0 -> 2
- net /GPIO8: track 0.00 -> 73.3 mm, vias 0 -> 2
- net /GPIO0: track 0.00 -> 72.0 mm, vias 0 -> 1
- net Net-(CHG1-A): track 0.00 -> 70.8 mm, vias 0 -> 1
- net /SENSOR_SCL: track 0.00 -> 69.0 mm, vias 0 -> 1
- net /US_SCL: track 0.00 -> 68.9 mm, vias 0 -> 1
- net /GPIO9: track 0.00 -> 67.8 mm, vias 0 -> 2
- net /GPIO1: track 0.00 -> 67.3 mm, vias 0 -> 1
- net /SENSOR_SDA: track 0.00 -> 65.8 mm, vias 0 -> 1
- net /US_SDA: track 0.00 -> 65.5 mm, vias 0 -> 1
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Other:
- board text added: "If USA good why USB?"
- board text added: "Put that back!"
- board text added: "Turn me on!"
- board text added: "U"
- board text added: "in duck."
- board text added: "w"
